File: kc1fsz-rx6.kicad_sch (KiCad schematic)
At the start: 2 parts, among them U1 SN74CBT3253

Commit message: Working
Parts:
- added C10, C14: 10u, symbol Device:C_Small
- added C11, C17: 10n, symbol Device:C_Small
- added C12, C13, C18, C19, C8, C9: 0.1u, symbol Device:C_Small
- added C15, C16, C6, C7: 4.7n, symbol Device:C_Small
- added C2: 2.2u, symbol Device:C_Small
- added C3, C4, C5: 33nF, symbol Device:C_Small
- added J1: Conn_Coaxial, symbol Connector:Conn_Coaxial
- added J2: Conn_01x07, symbol Connector_Generic:Conn_01x07
- added J3: Conn_01x04, symbol Connector_Generic:Conn_01x04
- added R1, R2: 10k, symbol Device:R_Small_US
- added R10, R17, R18, R19, R20, R9: 47, symbol Device:R_Small_US
- added R11, R8: 100k, symbol Device:R_Small_US
- added R12, R13, R6, R7: 470k, symbol Device:R_Small_US
- added R14, R3: 100, symbol Device:R_Small_US
- added R15, R16, R4, R5: 470, symbol Device:R_Small_US
- added TR1: TEZ0.5-D-2, Transformer_THT:Transformer_Breve_TEZ-22x24, symbol Transformer:TEZ0.5-D-2
- added U2, U3: LM4562, symbol Amplifier_Operational:LM4562
Connections:
- net GND: now also U1.1 (1~{OE}), U1.15 (2~{OE}), U1.8 (GND), C10.1, C14.1, C18.2, C19.2, C2.2, C3.2, C4.2, C5.2, J1.2 (Ext), J2.7 (Pin_7), J3.4 (Pin_4), R2.2, TR1.4, U2.4 (V-), U3.4 (V-)
- net CLK_I: now reaches U1.14 (S0)
- net CLK_I: now also R19.1
- net +5V: now reaches U1.16 (VCC)
- net +5V: now also C18.1, C19.1, J3.1 (Pin_1), R1.1, U2.8 (V+), U3.8 (V+)
- net CLK_Q: now reaches U1.2 (S1)
- net CLK_Q: now also R20.1
- net at U1.7 (1A): now also TR1.5
- net at U1.9 (2A): now also TR1.8
- net DET_0: no longer names the net of U1.13 (2B4), U1.6 (1B1)
- net DET_0: now also C5.1, C8.1
- net DET_180: no longer names the net of C1.1, U1.10 (2B1), U1.3 (1B4)
- net DET_180: now also C9.1
- net DET_270: no longer names the net of U1.12 (2B3), U1.5 (1B2)
- net DET_270: now also C13.1, C4.1
- net DET_90: no longer names the net of U1.11 (2B2), U1.4 (1B3)
- net DET_90: now also C12.1, C3.1
- new net: C15.1, R14.1, R15.1, U3.2 (-)
- new net: C15.2, R17.1, U3.1
- new net: J1.1 (In), TR1.1
- new net: C14.2, R11.2, R12.2, R13.1
- new net: C6.2, R9.1, U2.1
- new net: C6.1, R3.1, R4.1, U2.2 (-)
- new net: C8.2, R6.1, U2.3 (+)
- new net: C12.2, R13.2, U3.5 (+)
- new net: C2.1, R1.2, R2.1, TR1.6, TR1.7
- new net: C9.2, R7.2, U2.5 (+)
- new net: C7.1, R3.2, R5.1, U2.6 (-)
- new net: C7.2, R10.1, U2.7
- new net: C16.1, R14.2, R16.1, U3.6 (-)
- new net: C16.2, R18.1, U3.7
- new net: C13.2, R12.1, U3.3 (+)
- new net: C10.2, R6.2, R7.1, R8.2
- new net: J3.2 (Pin_2), R19.2
- new net: J3.3 (Pin_3), R20.2
- new net I_MINUS: C11.1, J2.2 (Pin_2), R10.2, R5.2
- new net I_PLUS: C11.2, J2.1 (Pin_1), R4.2, R9.2
- new net Q_MINUS: C17.1, J2.4 (Pin_4), R16.2, R18.2
- new net Q_PLUS: C17.2, J2.3 (Pin_3), R15.2, R17.2
- new net VCOML: J2.5 (Pin_5), R8.1
- new net VCOMR: J2.6 (Pin_6), R11.1
Other:
- moved on the sheet: C1, U1

Commit message: Initial PCB layout
Parts:
- removed J3: Conn_01x04, symbol Connector_Generic:Conn_01x04
- added H1, H2, H3, H4: MountingHole, MountingHole:MountingHole_3.5mm, symbol Mechanical:MountingHole
- added J3, J4: Conn_01x02, Connector_PinHeader_2.54mm:PinHeader_1x02_P2.54mm_Vertical, symbol Connector_Generic:Conn_01x02
- C1, C10, C11, C12, C13, C14, C15, C16, C17, C18, C19, C2, C3, C4, C5, C6, C7, C8, C9: footprint (none) -> Capacitor_SMD:C_0805_2012Metric_Pad1.18x1.45mm_HandSolder
- J1: footprint (none) -> Connector_Coaxial:SMA_Amphenol_901-144_Vertical
- J2: footprint (none) -> Connector_PinHeader_2.54mm:PinHeader_1x07_P2.54mm_Vertical
- R1, R10, R11, R12, R13, R14, R15, R16, R17, R18, R19, R2, R20, R3, R4, R5, R6, R7, R8, R9: footprint (none) -> Resistor_SMD:R_0805_2012Metric_Pad1.20x1.40mm_HandSolder
- TR1: value TEZ0.5-D-2 -> Trifilar FT37-43; footprint Transformer_THT:Transformer_Breve_TEZ-22x24 -> bruce-footprints:FT37-43 Trifilar
- U1: footprint (none) -> Package_SO:SOIC-16_3.9x9.9mm_P1.27mm
- U2, U3: footprint (none) -> Package_SO:SOIC-8_3.9x4.9mm_P1.27mm
Connections:
- net +5V: now also J3.1 (Pin_1)
- net GND: now also J3.2 (Pin_2)
- net Q_MINUS: now also J2.5 (Pin_5); no longer J2.4 (Pin_4)
- net Q_PLUS: now also J2.4 (Pin_4); no longer J2.3 (Pin_3)
- net VCOML: now also J2.3 (Pin_3); no longer J2.5 (Pin_5)
- net at R19.2: now also J4.1 (Pin_1)
- net at R20.2: now also J4.2 (Pin_2)
Other:
- moved on the sheet: R19, R20

Commit message: Layout complete
Parts:
- removed J4: Conn_01x02, Connector_PinHeader_2.54mm:PinHeader_1x02_P2.54mm_Vertical, symbol Connector_Generic:Conn_01x02
- added C20: 0.1u, Capacitor_SMD:C_0805_2012Metric_Pad1.18x1.45mm_HandSolder, symbol Device:C_Small
- added J4: Clock, Connector_PinHeader_2.54mm:PinHeader_1x04_P2.54mm_Vertical, symbol Connector_Generic:Conn_01x04
- added TP1, TP2: TestPoint, TestPoint:TestPoint_Pad_1.5x1.5mm, symbol Connector:TestPoint
- J3: value Conn_01x02 -> Power
Connections:
- net +5V: now also C20.1
- net GND: now also C20.2, J4.2 (Pin_2), J4.4 (Pin_4)
- net at R19.2: now also J4.1 (Pin_1)
- net at R20.2: now also J4.3 (Pin_3)
- net at TR1.5, U1.7 (1A): now also TP1.1
- net at TR1.8, U1.9 (2A): now also TP2.1
Other:
- moved on the sheet: R19, R20

Commit message: Working
Other:
- note added: "SOIC-16"
- note added: "SOIC-8"
Changed lines of the file:
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@@
+		)
+	)
+	(text "SOIC-8"
+		(exclude_from_sim no)
+		(at 235.458 37.084 0)
+		(effects
+			(font
+				(size 1.27 1.27)
+			)
+		)
+	)
+	(text "SOIC-16"
+		(exclude_from_sim no)
+		(at 113.03 77.724 0)
+		(effects
+			(font
+				(size 1.27 1.27)
+			)
+		)
+	)
+	(text "SOIC-8"
+		(exclude_from_sim no)
+		(at 235.204 94.234 0)
+		(effects
+			(font
+				(size 1.27 1.27)
+			)
 		)
 	)
